File: Hardware/HiBeam_4-pack_v02.sch (KiCad schematic (older format))
At the start: 16 parts, among them J1 5V, J2 CI, J3 DI, J4 GND, J5 CO, J6 DO, J7 5V, J8 GND, U1 APA102C, U2 APA102C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

Commit message: Fixes after double check.
Parts:
- added LOGO1: SFE_LOGO_NAME_FLAME.1_INCH, symbol SFE_LOGO_NAME_FLAME.1_INCH
- added LOGO2: OSHW-LOGOMINI, symbol OSHW-LOGOMINI
- C1, C2, C3, C4: value C -> 0.1uF
- U1, U2, U3, U4: footprint Pete:APA102 -> Pete:APA102_3
Other:
- note added: "1"
- note added: "Designed by Pete Dokter"
- note added: "HiBeam 4-pack"
- note added: "Released under the Creative Commons\nAttribution Share-Alike 4.0 License\nhttps://creativecommons.org/licenses/by-sa/4.0/"
Changed lines of the file:
@@
 LIBS:valves
 LIBS:apa102c
-LIBS:Hi-beam 4-pack v02-cache
+LIBS:SparkFun-Aesthetics
+LIBS:HiBeam_4-pack_v02-cache
 EELAYER 26 0
 EELAYER END
@@
 F 0 "U1" H 3700 3850 60  0000 C CNN
 F 1 "APA102C" H 3700 3450 60  0000 C CNN
-F 2 "Pete:APA102" H 3700 3650 60  0001 C CNN
+F 2 "Pete:APA102_3" H 3700 3650 60  0001 C CNN
 F 3 "" H 3700 3650 60  0001 C CNN
 	1    3700 3650
@@
 F 0 "U2" H 5200 3850 60  0000 C CNN
 F 1 "APA102C" H 5200 3450 60  0000 C CNN
-F 2 "Pete:APA102" H 5200 3650 60  0001 C CNN
+F 2 "Pete:APA102_3" H 5200 3650 60  0001 C CNN
 F 3 "" H 5200 3650 60  0001 C CNN
 	1    5200 3650
@@
 F 0 "U3" H 6700 3850 60  0000 C CNN
 F 1 "APA102C" H 6700 3450 60  0000 C CNN
-F 2 "Pete:APA102" H 6700 3650 60  0001 C CNN
+F 2 "Pete:APA102_3" H 6700 3650 60  0001 C CNN
 F 3 "" H 6700 3650 60  0001 C CNN
 	1    6700 3650
@@
 F 0 "U4" H 8200 3850 60  0000 C CNN
 F 1 "APA102C" H 8200 3450 60  0000 C CNN
-F 2 "Pete:APA102" H 8200 3650 60  0001 C CNN
+F 2 "Pete:APA102_3" H 8200 3650 60  0001 C CNN
 F 3 "" H 8200 3650 60  0001 C CNN
 	1    8200 3650
@@
 U 1 1 58F4E20E
 P 3700 3250
-F 0 "C1" H 3725 3350 50  0000 L CNN
-F 1 "C" H 3725 3150 50  0000 L CNN
+F 0 "C1" V 3654 3095 50  0000 L CNN
+F 1 "0.1uF" V 3645 3314 50  0000 L CNN
 F 2 "SparkFun-Capacitors:0603" H 3738 3100 50  0001 C CNN
 F 3 "" H 3700 3250 50  0000 C CNN
@@
 U 1 1 58F4E2CB
 P 5200 3250
-F 0 "C2" H 5225 3350 50  0000 L CNN
-F 1 "C" H 5225 3150 50  0000 L CNN
+F 0 "C2" V 5150 3085 50  0000 L CNN
+F 1 "0.1uF" V 5150 3300 50  0000 L CNN
 F 2 "SparkFun-Capacitors:0603" H 5238 3100 50  0001 C CNN
 F 3 "" H 5200 3250 50  0000 C CNN
@@
 U 1 1 58F4E386
 P 6700 3250
-F 0 "C3" H 6725 3350 50  0000 L CNN
-F 1 "C" H 6725 3150 50  0000 L CNN
+F 0 "C3" V 6652 3076 50  0000 L CNN
+F 1 "0.1uF" V 6650 3300 50  0000 L CNN
 F 2 "SparkFun-Capacitors:0603" H 6738 3100 50  0001 C CNN
 F 3 "" H 6700 3250 50  0000 C CNN
@@
 U 1 1 58F4E3F9
 P 8200 3250
-F 0 "C4" H 8225 3350 50  0000 L CNN
-F 1 "C" H 8225 3150 50  0000 L CNN
+F 0 "C4" V 8148 3083 50  0000 L CNN
+F 1 "0.1uF" V 8150 3300 50  0000 L CNN
 F 2 "SparkFun-Capacitors:0603" H 8238 3100 50  0001 C CNN
 F 3 "" H 8200 3250 50  0000 C CNN
@@
 $EndComp
 $Comp
-L +5V #PWR01
+L +5V #PWR4
 U 1 1 58F4E482
 P 4200 2950
-F 0 "#PWR01" H 4200 2800 50  0001 C CNN
+F 0 "#PWR4" H 4200 2800 50  0001 C CNN
 F 1 "+5V" H 4200 3090 50  0000 C CNN
 F 2 "" H 4200 2950 50  0000 C CNN
@@
 $EndComp
 $Comp
-L GND #PWR02
+L GND #PWR9
 U 1 1 58F4E4A6
 P 7700 4050
-F 0 "#PWR02" H 7700 3800 50  0001 C CNN
+F 0 "#PWR9" H 7700 3800 50  0001 C CNN
 F 1 "GND" H 7700 3900 50  0000 C CNN
 F 2 "" H 7700 4050 50  0000 C CNN
@@
 F 1 "DO" H 9750 3950 50  0000 C CNN
 F 2 "Pete:solder_pad_2" H 9750 3850 50  0001 C CNN
-F 3 "" H 9750 3850 50  0000 C CNN
+F 3 "" H 9750 3850 50  0001 C CNN
 	1    9750 3850
 	1    0    0    -1
 $EndComp
 $Comp
-L +5V #PWR03
+L +5V #PWR1
 U 1 1 58F4FD7D
 P 2150 4550
-F 0 "#PWR03" H 2150 4400 50  0001 C CNN
+F 0 "#PWR1" H 2150 4400 50  0001 C CNN
 F 1 "+5V" H 2150 4690 50  0000 C CNN
 F 2 "" H 2150 4550 50  0000 C CNN
@@
 $EndComp
 $Comp
-L GND #PWR04
+L GND #PWR2
 U 1 1 58F4FDE5
 P 2150 5800
-F 0 "#PWR04" H 2150 5550 50  0001 C CNN
+F 0 "#PWR2" H 2150 5550 50  0001 C CNN
 F 1 "GND" H 2150 5650 50  0000 C CNN
 F 2 "" H 2150 5800 50  0000 C CNN
@@
 Wire Wire Line
 	3550 3250 3200 3250
-Text Notes 10600 7650 0    60   ~ 12
+Text Notes 10600 7650 0    60   ~ 0
 v02
-Text Notes 8200 7650 0    60   ~ 12
+Text Notes 8200 7650 0    60   ~ 0
 5/8/17
 $Comp
@@
 Connection ~ 2150 5650
 $Comp
-L GND #PWR?
+L GND #PWR7
 U 1 1 591B6A1C
 P 6200 4050
-F 0 "#PWR?" H 6200 3800 50  0001 C CNN
+F 0 "#PWR7" H 6200 3800 50  0001 C CNN
 F 1 "GND" H 6200 3900 50  0000 C CNN
 F 2 "" H 6200 4050 50  0000 C CNN
@@
 $EndComp
 $Comp
-L GND #PWR?
+L GND #PWR5
 U 1 1 591B6A98
 P 4700 4050
-F 0 "#PWR?" H 4700 3800 50  0001 C CNN
+F 0 "#PWR5" H 4700 3800 50  0001 C CNN
 F 1 "GND" H 4700 3900 50  0000 C CNN
 F 2 "" H 4700 4050 50  0000 C CNN
@@
 $EndComp
 $Comp
-L GND #PWR?
+L GND #PWR3
 U 1 1 591B6C33
 P 3200 4050
-F 0 "#PWR?" H 3200 3800 50  0001 C CNN
+F 0 "#PWR3" H 3200 3800 50  0001 C CNN
 F 1 "GND" H 3200 3900 50  0000 C CNN
 F 2 "" H 3200 4050 50  0000 C CNN
@@
 $EndComp
 $Comp
-L +5V #PWR?
+L +5V #PWR6
 U 1 1 591B6CBE
 P 5700 2950
-F 0 "#PWR?" H 5700 2800 50  0001 C CNN
+F 0 "#PWR6" H 5700 2800 50  0001 C CNN
 F 1 "+5V" H 5700 3090 50  0000 C CNN
 F 2 "" H 5700 2950 50  0000 C CNN
@@
 $EndComp
 $Comp
-L +5V #PWR?
+L +5V #PWR8
 U 1 1 591B6D59
 P 7200 2950
-F 0 "#PWR?" H 7200 2800 50  0001 C CNN
+F 0 "#PWR8" H 7200 2800 50  0001 C CNN
 F 1 "+5V" H 7200 3090 50  0000 C CNN
 F 2 "" H 7200 2950 50  0000 C CNN
@@
 $EndComp
 $Comp
-L +5V #PWR?
+L +5V #PWR10
 U 1 1 591B6D84
 P 8700 2950
-F 0 "#PWR?" H 8700 2800 50  0001 C CNN
+F 0 "#PWR10" H 8700 2800 50  0001 C CNN
 F 1 "+5V" H 8700 3090 50  0000 C CNN
 F 2 "" H 8700 2950 50  0000 C CNN
@@
 Wire Wire Line
 	9200 3850 9550 3850
+Text Notes 7000 6934 0    79   ~ 0
+Released under the Creative Commons\nAttribution Share-Alike 4.0 License\nhttps://creativecommons.org/licenses/by-sa/4.0/
+Text Notes 7002 7088 0    79   ~ 0
+Designed by Pete Dokter
+Text Notes 7280 7246 0    61   ~ 0
+1
+Text Notes 7380 7244 0    61   ~ 0
+1
+Text Notes 7380 7496 0    61   ~ 0
+HiBeam 4-pack
+$Comp
+L SFE_LOGO_NAME_FLAME.1_INCH LOGO1
+U 1 1 591F24D0
+P 3550 7700
+F 0 "LOGO1" H 3550 7700 50  0001 C CNN
+F 1 "SFE_LOGO_NAME_FLAME.1_INCH" H 3550 7700 50  0001 C CNN
+F 2 "" H 3580 7850 20  0001 C CNN
+F 3 "" H 3550 7700 60  0001 C CNN
+	1    3550 7700
+	1    0    0    -1
+$EndComp
+$Comp
+L OSHW-LOGOMINI LOGO2
+U 1 1 591F2741
+P 6400 7250
+F 0 "LOGO2" H 6400 7250 50  0001 C CNN
+F 1 "OSHW-LOGOMINI" H 6400 7250 50  0001 C CNN
+F 2 "" H 6430 7400 20  0001 C CNN
+F 3 "" H 6400 7250 60  0001 C CNN
+	1    6400 7250
+	1    0    0    -1
+$EndComp
 $EndSCHEMATC
