File: Hardware/HiBeam_4-pack_v02.kicad_pcb (KiCad board)
At the start: 2 copper layers, 21.6 x 21.6 mm, 22 parts, among them J1 5V, J2 CI, J3 DI, J4 GND, J5 CO, J6 DO, J7 5V, J8 GND, U1 APA102C, U2 APA102C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

Commit message: Fixes after double check.
Parts:
- U1, U2, U3, U4: footprint Pete:APA102_2 -> Pete:APA102_3
Other:
- board text added: "1"
- board text added: "1/1"
- board text added: "2"
- board text added: "3"
- board text added: "4"
- board text added: "5/8/17"
- board text added: "HiBeam 4-pack"
- board text added: "Released under the Creative Commons Attribution Share-Alike 4.0 License https://creativecommons.org/licenses/by-sa/4.0/ Designed by Pete Dokter"

Commit message: Silk fixes.
Parts:
- ?: footprint SparkFun:SFE_LOGO_NAME_.1 -> Aesthetics:SFE_LOGO_NAME_FLAME_.1
- moved ? 1.15 mm to (151.6, 93.3)
