File: Hardware/Lumenati_4-pack.sch (KiCad schematic (older format))
At the start: 18 parts, among them J1 5V, J2 CI, J3 DI, J4 GND, J5 CO, J6 DO, J7 5V, J8 GND, U1 APA102C, U2 APA102C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

Commit message: Changed all the names to Lumenati, updated version to v10.
Other:
- note added: "Lumenati 4-pack"
- note added: "v10"
- note removed: "HiBeam 4-pack"
- note removed: "v02"
Changed lines of the file:
@@
 	3550 3250 3200 3250
 Text Notes 10600 7650 0    60   ~ 0
-v02
+v10
 Text Notes 8200 7650 0    60   ~ 0
 5/8/17
@@
 1
 Text Notes 7380 7496 0    61   ~ 0
-HiBeam 4-pack
+Lumenati 4-pack
 $Comp
 L SFE_LOGO_NAME_FLAME.1_INCH LOGO1

Commit message: Add fiducials to schematic.
Parts:
- added FD1, FD2: FIDUCIAL1X2, FIDUCIAL-1X2, symbol FIDUCIAL1X2
Changed lines of the file:
@@
 LIBS:contrib
 LIBS:valves
-LIBS:apa102c
+LIBS:SparkFun-Aesthetics - Copy
 LIBS:SparkFun-Aesthetics
-LIBS:HiBeam_4-pack_v02-cache
-EELAYER 26 0
+LIBS:SparkFun-Batteries
+LIBS:SparkFun-Boards
+LIBS:SparkFun-Capacitors
+LIBS:SparkFun-Clocks
+LIBS:SparkFun-Coils
+LIBS:SparkFun-Connectors
+LIBS:SparkFun-DiscreteSemi
+LIBS:SparkFun-Displays
+LIBS:SparkFun-Electromechanical
+LIBS:SparkFun-Fuses
+LIBS:SparkFun-GPS
+LIBS:SparkFun-Hardware
+LIBS:SparkFun-IC-Amplifiers
+LIBS:SparkFun-IC-Comms
+LIBS:SparkFun-IC-Conversion
+LIBS:SparkFun-IC-Logic
+LIBS:SparkFun-IC-Memory
+LIBS:SparkFun-IC-Microcontroller
+LIBS:SparkFun-IC-Power
+LIBS:SparkFun-IC-Special-Function
+LIBS:SparkFun-Jumpers
+LIBS:SparkFun-LED
+LIBS:SparkFun-PowerSymbols
+LIBS:SparkFun-Resistors
+LIBS:SparkFun-RF
+LIBS:SparkFun-Sensors
+LIBS:SparkFun-Switches
+LIBS:Lumenati_4-pack-cache
+EELAYER 25 0
 EELAYER END
 $Descr A4 11693 8268
@@
 	1    0    0    -1
 $EndComp
+$Comp
+L FIDUCIAL1X2 FD1
+U 1 1 5996EFF1
+P 11050 6200
+F 0 "FD1" H 11050 6300 45  0001 C CNN
+F 1 "FIDUCIAL1X2" H 11050 6100 45  0001 C CNN
+F 2 "FIDUCIAL-1X2" H 11050 6350 20  0001 C CNN
+F 3 "" H 11050 6200 60  0001 C CNN
+F 4 "XXX-00000" H 11050 6400 60  0001 C CNN "Field4"
+	1    11050 6200
+	1    0    0    -1
+$EndComp
+$Comp
+L FIDUCIAL1X2 FD2
+U 1 1 5996F030
+P 11050 6400
+F 0 "FD2" H 11050 6500 45  0001 C CNN
+F 1 "FIDUCIAL1X2" H 11050 6300 45  0001 C CNN
+F 2 "FIDUCIAL-1X2" H 11050 6550 20  0001 C CNN
+F 3 "" H 11050 6400 60  0001 C CNN
+F 4 "XXX-00000" H 11050 6600 60  0001 C CNN "Field4"
+	1    11050 6400
+	1    0    0    -1
+$EndComp
